File: eagle/main/beemos-master.sch (EAGLE design)
At the start: 50 parts, among them CON1 BAT, CON2 JACK_DC_BARREL, CON3 SPI, IC1 32U4, IC2 MCP73831T, IC3 MCP1703CB, IC4 DMP1045U, J1 RJ123.3, J10 RJ12STRAIGHT-I2C, J2 RJ123.3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

Commit message: Added modules to schematics
Parts:
- added U$6: SIM800L, SIM800L:SIM800L
- added U$7: MS5637, MS5637:MS5637
Other:
- note added: "Barometric pressure"
- note added: "GSM communication"
- note added: "Humidity"
- note added: "OneWire (Temperature)"
- note added: "Photoresistor"
- note added: "Rain sensor"
- note removed: "Temperature"
- moved on the sheet: C12, C13, LDR, R2

Commit message: Placed SIM800L module, added connections in schematic
Parts:
- removed C12: 10u, rcl:C-EUC0805K
- removed C13: 100nF, rcl:C-EUC0805K
- removed LDR: (no value), rcl:R-EU_0207/2V
- removed R2: 10k, rcl:R-EU_R0805
- removed U$7: MS5637, MS5637:MS5637
Connections:
- removed net SCL1: J1.1, J5.1
- removed net SCL2: J2.1
- removed net SCL3: J3.1, J6.1
- removed net SCL4: J4.1
- removed net SDA1: J1.6, J5.6
- removed net SDA2: J2.6
- removed net SDA3: J3.6, J6.6
- removed net SDA4: J4.6
- net 3.3V: now also U$6.RST
- net A5: no longer LDR.2, R2.2
- net D14: no longer C12.1, C13.1, R2.1
- net GND: now also U$6.GND; no longer C12.2, C13.2, LDR.1
- net RX: now also U$6.TXD
- net SCL: now also J1.1, J2.1, J3.1, J4.1, J5.1, J6.1
- net SDA: now also J1.6, J2.6, J3.6, J4.6, J5.6, J6.6
- net TX: now also U$6.RXD
- net VBAT1: now also U$6.VDD
Other:
- note removed: "Barometric pressure"
- note removed: "LDR"
- note removed: "Photoresistor"
